Commit message: [modify] 4wheel robot model

File: workspace/src/2D_Navigation_Stack/urdf/wheel.urdf.xacro (robot description, xacro)
@@ -40,5 +40,5 @@
       <kd  value="1.0" />
       <fdir1 value="1 0 0"/>
-      <material>Gazebo/Grey</material>
+      <material>Gazebo/Black</material>
       <turnGravityOff>false</turnGravityOff>
     </gazebo>

Commit message: [modify] hokuyo lidar

File: workspace/src/2D_Navigation_Stack/urdf/wheel.urdf.xacro (robot description, xacro)
@@ -55,8 +55,8 @@
       <type>transmission_interface/SimpleTransmission</type>
       <joint name="${fb}_${lr}_wheel_joint">
-        <hardwareInterface>EffortJointInterface</hardwareInterface>
+        <hardwareInterface>hardware_interface/EffortJointInterface</hardwareInterface>
       </joint>
       <actuator name="${fb}_${lr}_wheel_joint_motor">
-        <hardwareInterface>EffortJointInterface</hardwareInterface>
+        <hardwareInterface>hardware_interface/EffortJointInterface</hardwareInterface>
         <mechanicalReduction>1</mechanicalReduction>
       </actuator>

File: workspace/src/2D_Navigation_Stack/urdf/wheel_robot_base.urdf.xacro (robot description, xacro)
@@ -101,5 +101,5 @@
       <origin xyz="0 0 0" rpy="0 0 0" />
       <geometry>
-        <cylinder length="${hokuyo_size}" radius="${hokuyo_size}" />
+        <cylinder length="${hokuyo_size * 2}" radius="${hokuyo_size}" />
         <!--<box size="${hokuyo_size} ${hokuyo_size} ${hokuyo_size}"/>-->
       </geometry>
@@ -111,5 +111,6 @@
 <origin xyz="${base_radius - hokuyo_size/2} 0 ${base_height+hokuyo_size/4}" rpy="0 0 0" />
 -->
-    <origin xyz="${hokuyo_size/2} 0 ${0.15+hokuyo_size/4}" rpy="0 0 0" />
+    <!--<origin xyz="${hokuyo_size/2} 0 ${0.15+hokuyo_size/4}" rpy="0 0 0" />-->
+    <origin xyz="${hokuyo_size/2} 0 ${0.2+hokuyo_size/4}" rpy="0 0 0" />
     <parent link="base_link"/>
     <child link="hokuyo_link" />
@@ -120,13 +121,13 @@
     <sensor type="ray" name="head_hokuyo_sensor">
       <pose>${hokuyo_size/2} 0 0 0 0 0</pose>
-      <visualize>false</visualize>
+      <visualize>true</visualize>
       <update_rate>40</update_rate>
       <ray>
         <scan>
           <horizontal>
-            <samples>1024</samples>
+            <samples>4000</samples>
             <resolution>1</resolution>
-            <min_angle>-1.570796</min_angle>
-            <max_angle>1.570796</max_angle>
+            <min_angle>-3.14159</min_angle>
+            <max_angle>3.14159</max_angle>
           </horizontal>
         </scan>
