Commit message: [modify] 2D Navigation Stack

File: workspace/src/2D_Navigation_Stack/urdf/gmapbot.xacro (robot description, xacro)
@@ -145,12 +145,12 @@
  </joint>
   <!-- Camera joint -->
-  <joint name="camera_joint" type="fixed">
+  <!-- <joint name="camera_joint" type="fixed">
     <axis xyz="0 1 0" />
     <origin xyz="0.125 0 0.125" rpy="0 0 0"/>
     <parent link="base_link"/>
     <child link="camera_link"/>
-  </joint>
+  </joint> -->
   <!-- Camera -->
-  <link name="camera_link">
+  <!-- <link name="camera_link">
     <collision>
       <origin xyz="0 0 0" rpy="0 0 0"/>
@@ -173,14 +173,14 @@
       <inertia ixx="1e-6" ixy="0" ixz="0" iyy="1e-6" iyz="0" izz="1e-6" />
     </inertial>
-  </link>
+  </link> -->
   <!-- Hokuyo joint -->
-  <joint name="hokuyo_joint" type="fixed">
+  <!-- <joint name="hokuyo_joint" type="fixed">
     <origin xyz="0.125 0.05 0.125" rpy="0 0 0"/>
     <parent link="base_link"/>
     <axis xyz="0 1 0" />
     <child link="hokuyo_link"/>
-  </joint>
+  </joint> -->
   <!-- Hokuyo Laser -->
-  <link name="hokuyo_link">
+  <!-- <link name="hokuyo_link">
     <collision>
       <origin xyz="0 0 0" rpy="0 0 0"/>
@@ -226,6 +226,6 @@
 	      </plugin>
 	    </sensor>
-  	</gazebo>
-  <!-- Drive controller -->
+  	</gazebo> -->
+<!-- Drive controller -->
 <gazebo>
   <plugin name="skid_steer_drive_controller" filename="libgazebo_ros_skid_steer_drive.so">

File: workspace/src/2D_Navigation_Stack/urdf/wheel_robot_base.urdf.xacro (robot description, xacro)
@@ -95,11 +95,11 @@
   </gazebo>
   <!-- Hokuyo Laser scanner -->
-  <property name="hokuyo_size" value="0.1" />
+  <!-- property name="hokuyo_size" value="0.1" /> -->
   <!-- hokuyo -->
-  <link name="hokuyo_link">
+  <!-- <link name="hokuyo_link">
     <visual>
       <origin xyz="0 0 0" rpy="0 0 0" />
       <geometry>
-        <!--<box size="${hokuyo_size} ${hokuyo_size} ${hokuyo_size}"/>-->
+        <!-<box size="${hokuyo_size} ${hokuyo_size} ${hokuyo_size}"/>
         <cylinder length="${hokuyo_size * 2}" radius="${hokuyo_size}" />
       </geometry>
@@ -108,7 +108,4 @@
   </link>
   <joint name="hokuyo_joint" type="fixed">
-<!--
-<origin xyz="${base_radius - hokuyo_size/2} 0 ${base_height+hokuyo_size/4}" rpy="0 0 0" />
--->
     <origin xyz="${hokuyo_size/2} 0 ${0.2+hokuyo_size/4}" rpy="0 0 0" />
     <parent link="base_link"/>
@@ -142,4 +139,4 @@
       </plugin>
     </sensor>
-  </gazebo>
+  </gazebo> -->
 </robot>
